File: hw/baseline_project/baseline_project.kicad_sch (KiCad schematic)
At the start: 17 parts, among them J101 EXT_3V3, Q101 IRLD024PBF, SW101 UP, SW102 DOWN, SW103 LEFT, SW104 RIGHT, SW105 MODE, U101 EK-TM4C123GXL, U102 ESP8266-01/ESP-01, U103 Adafruit ST7735R

Commit message: SchematicDone
Parts:
- removed C101: 100nF, Capacitor_THT:C_Axial_L5.1mm_D3.1mm_P15.00mm_Horizontal, symbol Device:C_Small
- removed C103: 4.7uF, Capacitor_THT:CP_Axial_L10.0mm_D4.5mm_P15.00mm_Horizontal, symbol Device:C_Polarized_Small_US
- removed J101: EXT_3V3, Connector_Samtec_HPM_THT:Samtec_HPM-02-01-x-S_Straight_1x02_Pitch5.08mm, symbol Connector_Generic:Conn_01x02
- removed R101: 10k, Resistor_THT:R_Axial_DIN0411_L9.9mm_D3.6mm_P15.24mm_Horizontal, symbol Device:R_Small
- removed SW101: UP, Button_Switch_THT:SW_PUSH_6mm, symbol Switch:SW_Push
- removed SW102: DOWN, Button_Switch_THT:SW_PUSH_6mm, symbol Switch:SW_Push
- removed SW103: LEFT, Button_Switch_THT:SW_PUSH_6mm, symbol Switch:SW_Push
- removed SW104: RIGHT, Button_Switch_THT:SW_PUSH_6mm, symbol Switch:SW_Push
- removed SW105: MODE, Button_Switch_THT:SW_PUSH_6mm, symbol Switch:SW_Push
- removed U102: ESP8266-01/ESP-01, footprints:ai_thinker_ESP8266_01, symbol ai_thinker_ESP8266_01:ESP8266-01/ESP-01
- added C1, C2: 1u, Capacitor_SMD:C_1206_3216Metric, symbol Device:C_Small
- added D1, D2: LED, LED_THT:LED_D5.0mm, symbol Device:LED
- added IC1: AD5061BRJZ-1500RL7, footprints:SOT65P280X145-8N, symbol AD5061BRJZ-1500RL7:AD5061BRJZ-1500RL7
- added IC2: AD823ARZ, footprints:SOIC127P600X175-8N, symbol AD823ARZ:AD823ARZ
- added IC3: LP2950-33LPE3, TO127P419X482X788-3P, symbol LP2950-33LPE3:LP2950-33LPE3
- added J1: Logic, Connector_PinHeader_2.54mm:PinHeader_1x10_P2.54mm_Vertical, symbol Connector_Generic:Conn_01x10
- added J2: battery, Connector_PinHeader_2.54mm:PinHeader_1x02_P2.54mm_Vertical, symbol Connector_Generic:Conn_01x02
- added R1, R2, R3, R4, R5: R, Resistor_THT:R_Axial_DIN0411_L9.9mm_D3.6mm_P12.70mm_Horizontal, symbol Device:R
- added RV1: R_Potentiometer, Potentiometer_THT:Potentiometer_Bourns_PTA3043_Single_Slide, symbol Device:R_Potentiometer
- added SW1: UP, Button_Switch_THT:SW_PUSH_6mm, symbol Switch:SW_Push
- added TP1: gnd, TestPoint:TestPoint_Bridge_Pitch7.62mm_Drill1.3mm, symbol Connector:TestPoint
- added TP2: 3v3, TestPoint:TestPoint_Bridge_Pitch7.62mm_Drill1.3mm, symbol Connector:TestPoint
- added TP3: vbat, TestPoint:TestPoint_Bridge_Pitch7.62mm_Drill1.3mm, symbol Connector:TestPoint
- added TP4: dacOut, TestPoint:TestPoint_Bridge_Pitch7.62mm_Drill1.3mm, symbol Connector:TestPoint
- added TP5: spkr, TestPoint:TestPoint_Bridge_Pitch7.62mm_Drill1.3mm, symbol Connector:TestPoint
- added U1: LM4041LP-ADJ, Package_TO_SOT_THT:TO-92_Inline, symbol Reference_Voltage:LM4041LP-ADJ
Connections:
- net +3V3: now also C2.1, D2.2 (A), IC1.2 (VDD), IC2.8 (+VS), IC3.1 (OUTPUT), J1.9 (Pin_9), R3.1, RV1.1, SW1.2, TP2.1, U1.2 (K)
- net GND: now also C1.2, C2.2, IC1.5 (AGND), IC1.6 (DACGND), IC2.4 (-VS), IC3.2 (GND), J1.10 (Pin_10), J2.2 (Pin_2), R1.2, R2.2, R4.2, R5.2, RV1.3, TP1.1, U1.3 (A)
- net SDC_CS: now also J1.6 (Pin_6)
- net SPEAKER_GATE: now also IC2.1 (OUT1), IC2.2 (-IN1), TP5.1; no longer U101.J1_4 (PB1)
- net SW_MODE: now also R5.1, SW1.1
- net TFT_CS: now also J1.5 (Pin_5)
- net TFT_D/C: now also J1.7 (Pin_7)
- net TFT_MISO: now also J1.2 (Pin_2)
- net TFT_MOSI: now also J1.4 (Pin_4)
- net TFT_RST: now also J1.8 (Pin_8)
- net TFT_SCK: now also J1.3 (Pin_3)
- net DebugOut: now reaches U101.J2_2 (PB2)
- net DebugOut: now also D1.2 (A), J1.1 (Pin_1)
- net SS1_SCK: now reaches U101.J3_3 (PD0)
- net SS1_SCK: now also IC1.8 (SCLK)
- net SS1_FS: now reaches U101.J3_4 (PD1)
- net SS1_FS: now also IC1.7 (~{SYNC})
- net SS1_MOSI: now reaches U101.J3_6 (PD3)
- net SS1_MOSI: now also IC1.1 (DIN)
- net +5V renamed +BATT
- net +BATT: now also C1.1, IC3.3 (INPUT), J2.1 (Pin_1), TP3.1
- net SW_DOWN: no longer names the net of U101.J4_7 (PC7)
- net SW_LEFT: no longer names the net of U101.J4_6 (PC6)
- net SW_RIGHT: no longer names the net of U101.J4_5 (PC5)
- net SW_UP: no longer names the net of U101.J4_4 (PC4)
- net WIFI_IO2 renamed AIN
- net AIN: now also RV1.2
- net WIFI_RXD: no longer names the net of U101.J1_6 (PE5)
- net WIFI_TXD: no longer names the net of U101.J1_5 (PE4)
- net ~{WIFI_RST}: no longer names the net of U101.J3_7 (PE1)
- new net: D1.1 (K), R1.1
- new net: IC1.4 (VOUT), IC2.3 (+IN1), TP4.1
- new net: D2.1 (K), R2.1
- new net 1V5: IC1.3 (VREF), R3.2, R4.1, U1.1 (FB)
- no-connect marks 19 -> 26
Other:
- note removed: "AIN1"
- note removed: "I2C0_SCK"
- note removed: "SS1_FS"
- note removed: "SS1_MOSI"
- note removed: "SS1_SCK"
- moved on the sheet: C102, C104, D101, LS101, Q101, U103
